File: base_esp32.kicad_pcb (KiCad board)
At the start: 2 copper layers, 100 x 100 mm, 100 parts, among them J1 H_Src_raw, J10 S_IO, J11 H_KEYPAD, J12 S_KEYPAD, J13 BYPASS SRC 5V, J14 BYPASS SRC 3V3, J15 H_SERVO, J16 H_INA1, J17 H_BUZZER, J18 H_INB1, J19 H_IO34, J2 H_5V, J20 H_I2C, J21 S_I2C, J22 H_IO35, J23 H_INA2, J24 H_INB2, J25 H_IO36, J26 H_SPI, J27 S_SPI, J28 DTH11_V1, J29 DTH11_V2, J3 S_5V, J30 H_DTH11, J31 H_DS18B, J32 H_IO39, J33 TX_RX, J34 MOTOR, J35 H_TRIGGER, J36 H_IO33_OUT, J37 H_IO33, J38 ULTRASONIC, J39 H_IO15, J4 H_3V3_2, J40 H_IO15_OUT, J41 H_ECHO, J42 H_IO32, J43 H_IO32_OUT, J44 H_IO02, J45 H_IO02_OUT, J46 H_IO04, J47 H_IO04_OUT, J5 S_3V3_2, J6 H_GND, J7 S_GND, J8 Input Source, J9 H_IO, M1 Servo, SW1 SW_DIP_KEYPAD_1, SW2 SW_DIP_KEYPAD_2, SW3 ENABLE, SW4 BOOT, SW5 INPUT_D1, SW6 SW_DIP_INPUTS, SW7 INPUT_D2, SW8 Selector Input 1, SW9 Selector Input 2, U1 LM7805_TO220, U2 AMS1117, U3 ESP32-DevKitC, U4 AMS1117, U5 MX1508, U6 DS18B20, U7 LM35-LP

Commit message: add: router
Parts:
- added REF**: KiCad-Logo2_5mm_SilkScreen, Symbol:KiCad-Logo2_5mm_SilkScreen, F.Cu at (129.9, 102.6)
- added REF**: OSHW-Logo_7.5x8mm_SilkScreen, Symbol:OSHW-Logo_7.5x8mm_SilkScreen, F.Cu at (186.8, 136.0)
- added REF**: OSHW-Logo_7.5x8mm_SilkScreen, Symbol:OSHW-Logo_7.5x8mm_SilkScreen, B.Cu at (186.8, 136.0)
- added REF**: KiCad-Logo2_5mm_SilkScreen, Symbol:KiCad-Logo2_5mm_SilkScreen, B.Cu at (151.0, 57.8)
- moved J31 24.3 mm to (163.4, 134.5), turned to 0 degrees
- moved U6 17.9 mm to (164.7, 146.7)
- moved SW6 14.6 mm to (149.5, 140.1), turned to 90 degrees
- moved R5 12.1 mm to (167.3, 140.9), turned to 90 degrees
- moved J17 6.31 mm to (164.5, 113.4), turned to 90 degrees
- moved BZ1 6.21 mm to (156.9, 113.4)
- moved R10 5.55 mm to (147.9, 122.8)
- moved RV2 5.16 mm to (174.5, 145.8)
- moved SW8 5.16 mm to (179.5, 128.3)
- moved SW9 5.16 mm to (179.4, 134.9)
- moved J19 3.84 mm to (159.4, 144.4)
- moved J22 3.84 mm to (155.5, 144.4)
- moved J25 3.84 mm to (151.7, 144.4)
- moved J32 3.84 mm to (147.9, 144.4)
- moved R8 3.24 mm to (167.6, 122.8)
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Routing:
- net +5V: track 0.00 -> 436.9 mm, vias 0 -> 2
- net +3V3_1: track 0.00 -> 252.8 mm, vias 0 -> 3
- net /IO22: track 0.00 -> 201.8 mm, vias 0 -> 2
- net /DS18B: track 0.00 -> 148.2 mm, vias 0 -> 1
- net /IO02: track 0.00 -> 145.9 mm, vias 0 -> 1
- net /IO23: track 0.00 -> 145.9 mm, vias 0 -> 3
- net /IO21: track 0.00 -> 131.4 mm, vias 0 -> 3
- net /IO13: track 0.00 -> 128.1 mm, vias 0 -> 3
- net /IO12: track 0.00 -> 127.2 mm
- net /IO19: track 0.00 -> 119.0 mm, vias 0 -> 1
- net /IO04: track 0.00 -> 109.7 mm, vias 0 -> 2
- net /IO18: track 0.00 -> 108.5 mm, vias 0 -> 2
- net /IO05: track 0.00 -> 106.7 mm, vias 0 -> 4
- net /IO14: track 0.00 -> 99.4 mm
- net /IO17: track 0.00 -> 97.6 mm, vias 0 -> 3
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- added copper zone on B.Cu, net GND
- added copper zone on F.Cu, net GND
Other:
- board text added: "3V3_ESP32"
- board text added: "3V3_INT"
- board text added: "5V ESP32"
- board text added: "BRIDGE H"
- board text added: "BUZZER"
- board text added: "BYPASS"
- board text added: "ECHO/IO12"
- board text added: "IO02-IN2B"
- board text added: "IO02-OUT"
- board text added: "IO04"
- board text added: "IO04-OUT"
- board text added: "IO12K"
- board text added: "IO13K"
- board text added: "IO14K"
- board text added: "IO15-DS"
- board text added: "IO15-IN1B"
- board text added: "IO15-OUT"
- board text added: "IO16K"
- board text added: "IO17K"
- board text added: "IO25K"
- board text added: "IO26K"
- board text added: "IO27K"
- board text added: "IO32-IN2A"
- board text added: "IO32-OUT"
- board text added: "IO33-IN1A"
- board text added: "IO33-OUT"
- board text added: "IO36/D"
- board text added: "IO39/D"
- board text added: "OUTPUT VOLTAGE"
- board text added: "TRIGGER/IO13"
- board text added: "ULTRASONIC"
- board text added: "VCC"
- board text added: "VCC RAW"
- board text removed: "1"
- board text removed: "IN1A"
- board text removed: "IN1B"
- board text removed: "IN2A"
- board text removed: "IN2B"
- board text removed: "Input VCC"
- board text removed: "PUENTE H"
- board text removed: "ULTRASONICO"

Commit message: add: mark
Parts:
- added G***: LOGO, my_symbols:logo_x, F.Cu at (130.6, 100.6)
- added G***: LOGO, my_symbols:logo_x, B.Cu at (131.3, 100.8)
- added G***: LOGO, my_symbols:qr, B.Cu at (125.2, 80.2)
- moved REF** 50.9 mm to (167.9, 105.8)
- moved REF** 37.2 mm to (166.7, 107.7)
Routing:
- net /IO22: track 201.8 -> 150.0 mm, vias 2 -> 6
- net /IO23: track 145.9 -> 144.6 mm
- net GND: vias 24 -> 23
Other:
- board text added: "0.1600 mm / 0.1000 mm"
- board text added: "0.3000 mm"
- board text added: "1.6000 mm"
- board text added: "100.0000 mm x 100.0000 mm"
- board text added: "2"
- board text added: "BOARD CHARACTERISTICS"
- board text added: "Board Thickness:"
- board text added: "Board overall dimensions:"
- board text added: "Castellated pads:"
- board text added: "Copper Finish:"
- board text added: "Copper Layer Count:"
- board text added: "ECHO/ IO12"
- board text added: "Edge card connectors:"
- board text added: "IO00 -> BOOT IO01 -> TX IO02 -> DTH11 M2B IO03 -> RX IO04 -> - IO05 -> - IO06 -> X IO07 -> X IO08 -> X IO09 -> X IO10 -> X IO11 -> X IO12 -> K2 ECHO IO13 -> K1 TRIGGER IO14 -> K3 SERVO IO15 -> DS18B M1B IO16 -> K5 IO17 -> K6 IO18 -> - IO19 -> - IO20 -> X IO21 -> - IO22 -> - IO23 -> - IO24 -> X IO25 -> K7 IO26 -> K8 IO27 -> K4 IO28 -> X IO29 -> X IO30 -> X IO31 -> X IO32 -> BUZZER M2A IO33 -> M1A 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"
- board text added: "IO02-DTH11"
- board text added: "Impedance Control:"
- board text added: "Min hole diameter:"
- board text added: "Min track/spacing:"
- board text added: "No"
- board text added: "None"
- board text added: "Plated Board Edge:"
- board text added: "TRIGGER/ IO13"
- board text added: "x -> No connection - Free"
- board text removed: "ECHO/IO12"
- board text removed: "TRIGGER/IO13"
