File: base_esp32.kicad_pcb (KiCad board)
At the start: 2 copper layers, 100 x 100 mm, 107 parts, among them J1 H_Src_raw, J10 S_IO, J11 H_KEYPAD, J12 S_KEYPAD, J13 BYPASS SRC 5V, J14 BYPASS SRC 3V3, J15 H_SERVO, J16 H_INA1, J17 H_BUZZER, J18 H_INB1, J19 H_IO34, J2 H_5V, J20 H_I2C, J21 S_I2C, J22 H_IO35, J23 H_INA2, J24 H_INB2, J25 H_IO36, J26 H_SPI, J27 S_SPI, J28 DTH11_V1, J29 DTH11_V2, J3 S_5V, J30 H_DTH11, J31 H_DS18B, J32 H_IO39, J33 TX_RX, J34 MOTOR, J35 H_TRIGGER, J36 H_IO33_OUT, J37 H_IO33, J38 ULTRASONIC, J39 H_IO15, J4 H_3V3_2, J40 H_IO15_OUT, J41 H_ECHO, J42 H_IO32, J43 H_IO32_OUT, J44 H_IO02, J45 H_IO02_OUT, J46 H_IO04, J47 H_IO04_OUT, J5 S_3V3_2, J6 H_GND, J7 S_GND, J8 Input Source, J9 H_IO, M1 Servo, SW1 SW_DIP_KEYPAD_1, SW2 SW_DIP_KEYPAD_2, SW3 ENABLE, SW4 BOOT, SW5 INPUT_D1, SW6 SW_DIP_INPUTS, SW7 INPUT_D2, SW8 Selector Input 1, SW9 Selector Input 2, U1 LM7805_TO220, U2 AMS1117, U3 ESP32-DevKitC, U4 AMS1117, U5 MX1508, U6 DS18B20, U7 LM35-LP

Commit message: add: svg to fritzing in progress
Other:
- board text added: "JLCJLCJLCJLC"
- board text added: "KEYPAD"
- board text removed: "KEYBOARD"
Changed lines of the file:
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@@
+		)
+	)
+	(gr_text "JLCJLCJLCJLC"
+		(at 126.1364 60.5028 -0)
+		(layer "B.SilkS")
+		(effects
+			(font
+				(size 0.5 0.5)
+				(thickness 0.1)
+			)
+			(justify left bottom mirror)
+		)
+	)
+	(gr_text "KEYPAD"
+		(at 120.8024 145.517 -90)
+		(layer "B.SilkS")
+		(effects
+			(font
+				(size 0.8 0.8)
+				(thickness 0.15)
+			)
+			(justify mirror)
 		)
 	)
@@
 		)
 	)
-	(gr_text "KEYBOARD"
+	(gr_text "KEYPAD"
 		(at 120.8682 145.517 90)
 		(layer "F.SilkS")

Commit message: add: finish v0.1 devkit v4
Other:
- board text added: "DevKitV4"
Changed lines of the file:
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@@
 	(paper "A4")
 	(title_block
-		(title "Base ESP32")
+		(title "Base for ESP32 DevKit V4")
 		(date "2024-12-16")
 		(rev "v0.1")
@@
 			(sketchpadsonfab no)
 			(subtractmaskfromsilk yes)
-			(outputformat 1)
+			(outputformat 4)
 			(mirror no)
-			(drillshape 0)
+			(drillshape 2)
 			(scaleselection 1)
-			(outputdirectory "gerber/")
+			(outputdirectory "pcb/")
 		)
 	)
@@
 			(at 13.0302 -6.30936 180)
 			(layer "F.SilkS")
+			(hide yes)
 			(effects
 				(font
@@
 		)
 	)
+	(gr_text "DevKitV4"
+		(at 154.9908 105.5116 -0)
+		(layer "B.SilkS")
+		(effects
+			(font
+				(size 1 1)
+				(thickness 0.1)
+			)
+			(justify left bottom mirror)
+		)
+	)
 	(gr_text "5V\nESP32"
 		(at 116.7384 101.2952 0)
@@
 		)
 	)
-	(gr_text "IO00 -> BOOT\nIO01 -> TX\nIO02 -> DTH11 M2B\nIO03 -> RX\nIO04 -> -\nIO05 -> -\nIO06 -> X\nIO07 -> X\nIO08 -> X\nIO09 -> X\nIO10 -> X\nIO11 -> X\nIO12 -> K2 ECHO\nIO13 -> K1 TRIGGER\nIO14 -> K3 SERVO\nIO15 -> DS18B M1B\nIO16 -> K5\nIO17 -> K6\nIO18 -> -\nIO19 -> -\nIO20 -> X\nIO21 -> -\nIO22 -> -\nIO23 -> -\nIO24 -> X\nIO25 -> K7\nIO26 -> K8\nIO27 -> K4\nIO28 -> X\nIO29 -> X\nIO30 -> X\nIO31 -> X\nIO32 -> BUZZER M2A\nIO33 -> M1A\nIO34 -> POT_1/LDR\nIO35 -> POT_2/LM35\nIO36 -> -\nIO37 -> X\nIO38 -> X\nIO39 -> -"
+	(gr_text "IO00 -> BOOT\nIO01 -> TX\nIO02 -> DTH11 M2B\nIO03 -> RX\nIO04 -> -\nIO05 -> -\nIO06 -> X\nIO07 -> X\nIO08 -> X\nIO09 -> X\nIO10 -> X\nIO11 -> X\nIO12 -> K2 ECHO\nIO13 -> K1 TRIGGER\nIO14 -> K3 SERVO\nIO15 -> DS18B M1B\nIO16 -> K5\nIO17 -> K6\nIO18 -> -\nIO19 -> -\nIO20 -> X\nIO21 -> -\nIO22 -> -\nIO23 -> -\nIO24 -> X\nIO25 -> K7\nIO26 -> K8\nIO27 -> K4\nIO28 -> X\nIO29 -> X\nIO30 -> X\nIO31 -> X\nIO32 -> BUZZER M2A\nIO33 -> M1A\nIO34 -> POT_1/LDR\nIO35 -> POT_2/LM35\nIO36 -> DI VP\nIO37 -> X\nIO38 -> X\nIO39 -> DI VN"
 		(at 159.1564 103.378 0)
 		(layer "B.SilkS")
@@
 		)
 	)
-	(gr_text "IO00 -> BOOT\nIO01 -> TX\nIO02 -> DTH11 M2B\nIO03 -> RX\nIO04 -> -\nIO05 -> -\nIO06 -> X\nIO07 -> X\nIO08 -> X\nIO09 -> X\nIO10 -> X\nIO11 -> X\nIO12 -> K2 ECHO\nIO13 -> K1 TRIGGER\nIO14 -> K3 SERVO\nIO15 -> DS18B M1B\nIO16 -> K5\nIO17 -> K6\nIO18 -> -\nIO19 -> -\nIO20 -> X\nIO21 -> -\nIO22 -> -\nIO23 -> -\nIO24 -> X\nIO25 -> K7\nIO26 -> K8\nIO27 -> K4\nIO28 -> X\nIO29 -> X\nIO30 -> X\nIO31 -> X\nIO32 -> BUZZER M2A\nIO33 -> M1A\nIO34 -> POT_1/LDR\nIO35 -> POT_2/LM35\nIO36 -> -\nIO37 -> X\nIO38 -> X\nIO39 -> -"
+	(gr_text "IO00 -> BOOT\nIO01 -> TX\nIO02 -> DTH11 M2B\nIO03 -> RX\nIO04 -> -\nIO05 -> -\nIO06 -> X\nIO07 -> X\nIO08 -> X\nIO09 -> X\nIO10 -> X\nIO11 -> X\nIO12 -> K2 ECHO\nIO13 -> K1 TRIGGER\nIO14 -> K3 SERVO\nIO15 -> DS18B M1B\nIO16 -> K5\nIO17 -> K6\nIO18 -> -\nIO19 -> -\nIO20 -> X\nIO21 -> -\nIO22 -> -\nIO23 -> -\nIO24 -> X\nIO25 -> K7\nIO26 -> K8\nIO27 -> K4\nIO28 -> X\nIO29 -> X\nIO30 -> X\nIO31 -> X\nIO32 -> BUZZER M2A\nIO33 -> M1A\nIO34 -> POT_1/LDR\nIO35 -> POT_2/LM35\nIO36 -> DI VP\nIO37 -> X\nIO38 -> X\nIO39 -> DI VN"
 		(at 143.3068 103.378 0)
 		(layer "F.SilkS")
@@
 				(thickness 0.1)
 			)
+			(justify left bottom)
+		)
+	)
+	(gr_text "DevKitV4"
+		(at 148.3868 105.5116 0)
+		(layer "F.SilkS")
+		(effects
+			(font
+				(size 1 1)
+				(thickness 0.1)
+			)
