File: base_esp32.kicad_sch (KiCad schematic)
At the start: 100 parts, among them J1 H_Src_raw, J10 S_IO, J11 H_KEYPAD, J12 S_KEYPAD, J13 BYPASS SRC 5V, J14 BYPASS SRC 3V3, J15 H_SERVO, J16 H_INA1, J17 H_BUZZER, J18 H_INB1, J19 H_IO34, J2 H_5V, J20 H_I2C, J21 S_I2C, J22 H_IO35, J23 H_INA2, J24 H_INB2, J25 H_IO36, J26 H_SPI, J27 S_SPI, J28 DTH11_V1, J29 DTH11_V2, J3 S_5V, J30 H_DTH11, J31 H_DS18B, J32 H_IO39, J33 TX_RX, J34 MOTOR, J35 H_TRIGGER, J36 H_IO33_OUT, J37 H_IO33, J38 ULTRASONIC, J39 H_IO15, J4 H_3V3_2, J40 H_IO15_OUT, J41 H_ECHO, J42 H_IO32, J43 H_IO32_OUT, J44 H_IO02, J45 H_IO02_OUT, J46 H_IO04, J47 H_IO04_OUT, J5 S_3V3_2, J6 H_GND, J7 S_GND, J8 Input Source, J9 H_IO, M1 Servo, SW1 SW_DIP_KEYPAD_1, SW2 SW_DIP_KEYPAD_2, SW3 ENABLE, SW4 BOOT, SW5 INPUT_D1, SW6 SW_DIP_INPUTS, SW7 INPUT_D2, SW8 Selector Input 1, SW9 Selector Input 2, U1 LM7805_TO220, U2 AMS1117, U3 ESP32-DevKitC, U4 AMS1117, U5 MX1508, U6 DS18B20, U7 LM35-LP

Commit message: add: mark
Parts:
- U2, U4: LCSC Part (none) -> C22458961

Commit message: add: finish v0.1 devkit v4
Other:
- title: Base for ESP32 -> Base for ESP32 DevKit V4
Changed lines of the file:
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@@
 	(paper "A4")
 	(title_block
-		(title "Base for ESP32")
+		(title "Base for ESP32 DevKit V4")
 		(date "2024-11-27")
 		(rev "0.1")
@@
 		)
 	)
+	(polyline
+		(pts
+			(xy 265.35 161.29) (xy 265.35 161.29)
+		)
+		(stroke
+			(width -0.0001)
+			(type solid)
+		)
+	)
 	(wire
 		(pts
@@
 		)
 	)
-	(polyline
-		(pts
-			(xy 265.35 161.29) (xy 265.35 161.29)
-		)
-		(stroke
-			(width -0.0001)
-			(type solid)
-		)
-		(fill
-			(type color)
-			(color 26 26 26 1)
-		)
-	)
